File: schematic/RetroGameCard/retroGameCard/retroGameCard.kicad_sch (KiCad schematic)
At the start: 34 parts, among them IC1 STM32C562KET6, J2 Conn_01x04_Pin, J3 USB_C_Receptacle_USB2.0_16P, SW1 SW_Slide_DPDT, SW2 SW_SPDT, SW3 SW_Push, SW4 SW_Push, SW5 SW_Push, SW6 SW_Push, SW7 SW_Push, U1 MCP73831-2-OT, U2 AP2112K-3.3, U3 DM-OLED096-636

Commit message: added mounting holes in schematic
Parts:
- added H1, H2, H3, H4: MountingHole, MountingHole:MountingHole_3.2mm_M3, symbol Mechanical:MountingHole
