File: schematic/RetroGameCard/retroGameCard/_restore_backup_2026-07-12T14-25-27-690/retroGameCard.kicad_pcb (KiCad board)
At the start: 2 copper layers, 52.5 x 85 mm, 38 parts, among them IC1 STM32C562KET6, J2 Conn_01x04_Pin, J3 USB_C_Receptacle_USB2.0_16P, SW1 SW_Slide_DPDT, SW2 SW_SPDT, SW3 SW_Push, SW4 SW_Push, SW5 SW_Push, SW6 SW_Push, SW7 SW_Push, U1 MCP73831-2-OT, U2 AP2112K-3.3, U3 DM-OLED096-636

Commit message: finished board - ready to be manufacture
Parts:
- added G***: LOGO, LOGO, F.Cu at (230.7, 62.6)
Routing:
- net GND: track 98.0 -> 98.7 mm
Other:
- board text added: "12.07.2026"
- board text added: "BOOT"
- board text added: "Youtube.com/ @AlwaysIterate"
- board text removed: "(symbol "LOGO" (pin_names (offset 1.016)) (in_bom yes) (on_board yes) (property "Reference" "#G" (at 0 6.86711 0) (effects (font (size 1.27 1.27)) hide) ) (property "Value" "LOGO" (at 0 -6.86711 0) (effects (font (size 1.27 1.27)) hide) ) (property "Footprint" "" (at 0 0 0) (effects (font (size 1.27 1.27)) hide) ) (property "Datasheet" "" (at 0 0 0) (effects (font (size 1.27 1.27)) hide) ) (symbo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"
- board text removed: "Youtube.com/@AlwaysIterate"
